File: Conmutador_antenas_1x6.kicad_pcb (KiCad board)
At the start: 0 parts

Commit message: Finished board layout
0.1.0
Parts:
- added A1: RaspberryPi_Pico_W, Cfootprints:Pi pico 2w pin, F.Cu at (45.3, 128.4)
- added C1: 22nF, Capacitor_THT:C_Disc_D5.0mm_W2.5mm_P5.00mm, F.Cu at (18.4, 137.7)
- added C2: 22nF, Capacitor_THT:C_Disc_D5.0mm_W2.5mm_P5.00mm, F.Cu at (18.4, 132.7)
- added D1: 1n4007, Diode_THT:D_DO-41_SOD81_P7.62mm_Horizontal, F.Cu at (144.1, 82.0)
- added D10: LED, LED_THT:LED_D3.0mm, F.Cu at (227.1, 91.9)
- added D11: LED, LED_THT:LED_D3.0mm, F.Cu at (253.1, 92.0)
- added D12: LED, LED_THT:LED_D3.0mm, F.Cu at (279.1, 92.0)
- added D2: 1n4007, Diode_THT:D_DO-41_SOD81_P7.62mm_Horizontal, F.Cu at (169.8, 82.1)
- added D3: 1n4007, Diode_THT:D_DO-41_SOD81_P7.62mm_Horizontal, F.Cu at (195.8, 82.1)
- added D4: 1n4007, Diode_THT:D_DO-41_SOD81_P7.62mm_Horizontal, F.Cu at (221.8, 82.1)
- added D5: 1n4007, Diode_THT:D_DO-41_SOD81_P7.62mm_Horizontal, F.Cu at (247.7, 82.1)
- added D6: 1n4007, Diode_THT:D_DO-41_SOD81_P7.62mm_Horizontal, F.Cu at (273.8, 82.2)
- added D7: LED, LED_THT:LED_D3.0mm, F.Cu at (149.3, 91.9)
- added D8: LED, LED_THT:LED_D3.0mm, F.Cu at (175.1, 92.0)
- added D9: LED, LED_THT:LED_D3.0mm, F.Cu at (201.1, 91.9)
- added J1: Conn_Coaxial, Cfootprints:SO-239, F.Cu at (140.3, 127.5)
- added J10: Conn_01x20, Connector_PinHeader_2.54mm:PinHeader_1x20_P2.54mm_Vertical, F.Cu at (49.5, 128.4)
- added J11: Conn_01x20, Connector_PinHeader_2.54mm:PinHeader_1x20_P2.54mm_Vertical, F.Cu at (23.9, 128.4)
- added J12: Screw_Terminal_01x02, TerminalBlock_Phoenix:TerminalBlock_Phoenix_MKDS-1,5-2-5.08_1x02_P5.08mm_Horizontal, F.Cu at (62.9, 142.0)
- added J13: Conn_01x02, Connector_PinHeader_2.54mm:PinHeader_1x02_P2.54mm_Vertical, F.Cu at (66.4, 130.9)
- added J14: Conn_01x02, Connector_PinHeader_2.54mm:PinHeader_1x02_P2.54mm_Vertical, F.Cu at (66.4, 126.3)
- added J15: Screw_Terminal_01x02, TerminalBlock_Phoenix:TerminalBlock_Phoenix_MKDS-1,5-2-5.08_1x02_P5.08mm_Horizontal, F.Cu at (50.9, 142.0)
- added J16: Conn_01x07, Connector_PinHeader_2.54mm:PinHeader_1x07_P2.54mm_Vertical, F.Cu at (53.4, 123.2)
- added J17: Conn_01x04, Connector_PinHeader_2.54mm:PinHeader_1x04_P2.54mm_Vertical, F.Cu at (19.4, 77.6)
- added J2: Conn_Coaxial, Cfootprints:SO-239, F.Cu at (166.1, 127.5)
- added J3: Conn_Coaxial, Cfootprints:SO-239, F.Cu at (192.1, 127.5)
- added J4: Screw_Terminal_01x07, TerminalBlock_Phoenix:TerminalBlock_Phoenix_MKDS-1,5-7-5.08_1x07_P5.08mm_Horizontal, F.Cu at (105.8, 71.9)
- added J5: Conn_Coaxial, Cfootprints:SO-239, F.Cu at (114.1, 127.5)
- added J6: Conn_Coaxial, Cfootprints:SO-239, F.Cu at (218.1, 127.5)
- added J7: Conn_Coaxial, Cfootprints:SO-239, F.Cu at (244.1, 127.5)
- added J8: Conn_Coaxial, Cfootprints:SO-239, F.Cu at (270.1, 127.5)
- added J9: Screw_Terminal_01x08, TerminalBlock_Phoenix:TerminalBlock_Phoenix_MKDS-1,5-8-5.08_1x08_P5.08mm_Horizontal, F.Cu at (85.8, 107.5)
- added K1: ~, Footprints:Relay_DPDT_Schrack-RT2-FormC_RM5mm, F.Cu at (136.4, 86.5)
- added K2: ~, Footprints:Relay_DPDT_Schrack-RT2-FormC_RM5mm, F.Cu at (162.2, 86.7)
- added K3: ~, Footprints:Relay_DPDT_Schrack-RT2-FormC_RM5mm, F.Cu at (188.2, 86.7)
- added K4: ~, Footprints:Relay_DPDT_Schrack-RT2-FormC_RM5mm, F.Cu at (214.2, 86.7)
- added K5: ~, Footprints:Relay_DPDT_Schrack-RT2-FormC_RM5mm, F.Cu at (240.2, 86.7)
- added K6: ~, Footprints:Relay_DPDT_Schrack-RT2-FormC_RM5mm, F.Cu at (266.2, 86.7)
- added R1: 1k, Resistor_THT:R_Axial_DIN0204_L3.6mm_D1.6mm_P5.08mm_Horizontal, F.Cu at (149.3, 82.0)
- added R10: 470R, Resistor_THT:R_Axial_DIN0204_L3.6mm_D1.6mm_P7.62mm_Horizontal, F.Cu at (59.1, 89.8)
- added R11: 470R, Resistor_THT:R_Axial_DIN0204_L3.6mm_D1.6mm_P7.62mm_Horizontal, F.Cu at (59.1, 80.8)
- added R12: 470R, Resistor_THT:R_Axial_DIN0204_L3.6mm_D1.6mm_P7.62mm_Horizontal, F.Cu at (59.1, 71.8)
- added R2: 1k, Resistor_THT:R_Axial_DIN0204_L3.6mm_D1.6mm_P5.08mm_Horizontal, F.Cu at (175.1, 82.1)
- added R3: 1k, Resistor_THT:R_Axial_DIN0204_L3.6mm_D1.6mm_P5.08mm_Horizontal, F.Cu at (201.1, 82.1)
- added R4: 1k, Resistor_THT:R_Axial_DIN0204_L3.6mm_D1.6mm_P5.08mm_Horizontal, F.Cu at (227.1, 82.1)
- added R5: 1k, Resistor_THT:R_Axial_DIN0204_L3.6mm_D1.6mm_P5.08mm_Horizontal, F.Cu at (253.1, 82.1)
- added R6: 1k, Resistor_THT:R_Axial_DIN0204_L3.6mm_D1.6mm_P5.08mm_Horizontal, F.Cu at (279.1, 82.2)
- added R7: 470R, Resistor_THT:R_Axial_DIN0204_L3.6mm_D1.6mm_P7.62mm_Horizontal, F.Cu at (59.1, 116.8)
- added R8: 470R, Resistor_THT:R_Axial_DIN0204_L3.6mm_D1.6mm_P7.62mm_Horizontal, F.Cu at (59.0, 107.7)
- added R9: 470R, Resistor_THT:R_Axial_DIN0204_L3.6mm_D1.6mm_P7.62mm_Horizontal, F.Cu at (59.1, 98.8)
- added REF**: MountingHole_3.2mm_M3, MountingHole:MountingHole_3.2mm_M3, F.Cu at (13.5, 63.9)
- added REF**: MountingHole_3.2mm_M3, MountingHole:MountingHole_3.2mm_M3, F.Cu at (192.5, 63.9)
- added REF**: MountingHole_3.2mm_M3, MountingHole:MountingHole_3.2mm_M3, F.Cu at (192.0, 146.0)
- added REF**: MountingHole_3.2mm_M3, MountingHole:MountingHole_3.2mm_M3, F.Cu at (105.0, 146.0)
- added REF**: MountingHole_3.2mm_M3, MountingHole:MountingHole_3.2mm_M3, F.Cu at (86.0, 64.0)
- added REF**: MountingHole_3.2mm_M3, MountingHole:MountingHole_3.2mm_M3, F.Cu at (13.5, 145.9)
- added REF**: MountingHole_3.2mm_M3, MountingHole:MountingHole_3.2mm_M3, F.Cu at (285.5, 145.9)
- added REF**: MountingHole_3.2mm_M3, MountingHole:MountingHole_3.2mm_M3, F.Cu at (85.5, 146.1)
- added REF**: MountingHole_3.2mm_M3, MountingHole:MountingHole_3.2mm_M3, F.Cu at (285.5, 63.9)
- added REF**: MountingHole_3.2mm_M3, MountingHole:MountingHole_3.2mm_M3, F.Cu at (105.5, 63.9)
- added U1: 4N25, Package_DIP:DIP-6_W7.62mm, F.Cu at (69.2, 116.8)
- added U2: 4N25, Package_DIP:DIP-6_W7.62mm, F.Cu at (69.2, 107.7)
- added U3: 4N25, Package_DIP:DIP-6_W7.62mm, F.Cu at (69.2, 98.7)
- added U4: 4N25, Package_DIP:DIP-6_W7.62mm, F.Cu at (69.2, 89.7)
- added U5: 4N25, Package_DIP:DIP-6_W7.62mm, F.Cu at (69.2, 80.7)
- added U6: 4N25, Package_DIP:DIP-6_W7.62mm, F.Cu at (69.2, 71.7)
- added U7: LM7805_TO220, Package_TO_SOT_THT:TO-220-3_Vertical, F.Cu at (15.3, 137.8)
Routing:
- net /Controlador/OUT_{6}: track 0.00 -> 224.4 mm
- net /Controlador/OUT_{5}: track 0.00 -> 201.7 mm
- net /Controlador/OUT_{4}: track 0.00 -> 181.2 mm
- net /Reles/RF_{IN}: track 0.00 -> 172.7 mm
- net /Controlador/OUT_{3}: track 0.00 -> 160.0 mm
- net /Controlador/OUT_{2}: track 0.00 -> 139.2 mm
- net /Controlador/OUT_{1}: track 0.00 -> 118.7 mm
- net +12V: track 0.00 -> 118.5 mm
- net +5V: track 0.00 -> 74.5 mm
- net GND1: track 0.00 -> 63.5 mm
- net +12C: track 0.00 -> 62.1 mm
- net 3V3: track 0.00 -> 52.0 mm
- net GND: track 0.00 -> 39.7 mm
- net /Controlador/GP10: track 0.00 -> 32.7 mm
- net /Reles/RF_{antena-1}: track 0.00 -> 28.1 mm
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- added copper zone on B.Cu, net GND
- added copper zone on F.Cu, net GND
- added copper zone on B.Cu, net GND1
- added copper zone on F.Cu, net GND1
Other:
- board outline added: 280 x 90 mm
- copper layers 0 -> 2
- board text added: "-"
- board text added: "0.1.0"
- board text added: "1"
- board text added: "12V"
- board text added: "1x6"
- board text added: "2"
- board text added: "3"
- board text added: "3V3"
- board text added: "4"
- board text added: "5"
- board text added: "5V"
- board text added: "6"
- board text added: "Antena GND"
- board text added: "CS"
- board text added: "Conmutador"
- board text added: "Conmutador de antenas"
- board text added: "Controlador"
- board text added: "DC"
- board text added: "Diseñado por winsrrow"
- board text added: "GND"
- board text added: "GND-1"
- board text added: "I2C"
- board text added: "IN"
- board text added: "Opciones:"
- board text added: "Puentes alimentación"
- board text added: "Puertos:"
- board text added: "RES"
- board text added: "SCK"
- board text added: "SCL"
- board text added: "SDA"
- board text added: "SPI"
- board text added: "USB KEEPOUT"
- board text added: "VCC"
- board text added: "VCC-1"
- board text added: "Versión:"
- board text added: "WIFI"
