File: Controlador.kicad_sch (KiCad schematic)
At the start: 21 parts, among them J10 Conn_01x20, J11 Conn_01x20, J12 Conn_01x07, J13 Screw_Terminal_01x02, J9 Screw_Terminal_01x08, U1 4N25, U2 4N25, U3 4N25, U4 4N25, U5 4N25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

Commit message: Finished board layout
0.1.0
Parts:
- added J12: Screw_Terminal_01x02, TerminalBlock_Phoenix:TerminalBlock_Phoenix_MKDS-1,5-2-5.08_1x02_P5.08mm_Horizontal, symbol CA16:Screw_Terminal_01x02
- added J13, J14: Conn_01x02, Connector_PinHeader_2.54mm:PinHeader_1x02_P2.54mm_Vertical, symbol Connector_Generic:Conn_01x02
- added J17: Conn_01x04, Connector_PinHeader_2.54mm:PinHeader_1x04_P2.54mm_Vertical, symbol Connector_Generic:Conn_01x04
- A1: footprint Module:RaspberryPi_Pico_W_SMD_HandSolder -> Cfootprints:Pi pico 2w pin; symbol CSym:RaspberryPi_Pico_2W_Debug -> CA16:RaspberryPi_Pico_2W_Debug
- C1: renamed from C7; symbol Device:C_Polarized_US -> CA16:C_Polarized_US
- C2: renamed from C8; symbol Device:C_Polarized_US -> CA16:C_Polarized_US
- J10: footprint (none) -> Connector_PinHeader_2.54mm:PinHeader_1x20_P2.54mm_Vertical; symbol Connector_Generic:Conn_01x20 -> CA16:Conn_01x20; Use (none) -> Izquierda; use Izquierda -> (none)
- J11: footprint (none) -> Connector_PinHeader_2.54mm:PinHeader_1x20_P2.54mm_Vertical; symbol Connector_Generic:Conn_01x20 -> CA16:Conn_01x20; Use (none) -> Derecha; use Derecha -> (none)
- J15: renamed from J13; symbol Connector:Screw_Terminal_01x02 -> CA16:Screw_Terminal_01x02
- J16: renamed from J12; footprint (none) -> Connector_PinHeader_2.54mm:PinHeader_1x07_P2.54mm_Vertical; symbol Connector_Generic:Conn_01x07 -> CA16:Conn_01x07; Use (none) -> OLED SPI; use OLED SPI -> (none)
- J9: symbol Connector:Screw_Terminal_01x08 -> CA16:Screw_Terminal_01x08
- R10, R11, R12, R7, R8, R9: symbol Device:R -> CA16:R
- U1, U2, U3, U4, U5, U6: symbol Isolator:4N25 -> CA16:4N25
- U7: symbol Regulator_Linear:LM7805_TO220 -> CA16:LM7805_TO220
Connections:
- net +12V: now also J9.1 (Pin_1), J12.2 (Pin_2), J13.1 (Pin_1); no longer C1.1, J15.2 (Pin_2), J9.8 (Pin_8), U7.1 (VI)
- net +5V: now also J17.1 (Pin_1)
- net GND: now also J14.2 (Pin_2), J17.4 (Pin_4); no longer A1.D2 (GND), J9.1 (Pin_1)
- net GP16: now also J17.2 (Pin_2)
- net GP17: now also J17.3 (Pin_3)
- net OUT_{1}: now also J9.2 (Pin_2); no longer J9.7 (Pin_7)
- net OUT_{2}: now also J9.3 (Pin_3); no longer J9.6 (Pin_6)
- net OUT_{3}: now also J9.4 (Pin_4); no longer J9.5 (Pin_5)
- net OUT_{4}: now also J9.5 (Pin_5); no longer J9.4 (Pin_4)
- net OUT_{5}: now also J9.6 (Pin_6); no longer J9.3 (Pin_3)
- net OUT_{6}: now also J9.7 (Pin_7); no longer J9.2 (Pin_2)
- new net +12C: C1.1, J13.2 (Pin_2), J15.2 (Pin_2), U7.1 (VI)
- new net GND1: J12.1 (Pin_1), J14.1 (Pin_1), J9.8 (Pin_8)
- no-connect marks 0 -> 11
Other:
- note added: "Controlador"
- note added: "Drivers"
- note added: "SPI"
- moved on the sheet: J15
