File: Reles.kicad_sch (KiCad schematic)
At the start: 38 parts, among them J1 Conn_Coaxial, J2 Screw_Terminal_01x07, J3 Conn_Coaxial, J4 Conn_Coaxial, J5 Conn_Coaxial, J6 Conn_Coaxial, J7 Conn_Coaxial, J8 Conn_Coaxial

Commit message: Finished board layout
0.1.0
Parts:
- removed C1, C2, C3, C4, C5, C6: 100nF, Capacitor_THT:C_Disc_D5.0mm_W2.5mm_P2.50mm, symbol schematic:C
- removed J3, J4, J7, J8: Conn_Coaxial, Footprints:PL_PanelMount, symbol schematic:Conn_Coaxial
- removed K2, K3, K4: ~, Footprints:Relay_DPDT_Schrack-RT2-FormC_RM5mm, symbol schematic:Rele_2Conm
- added J2, J3, J6, J8: Conn_Coaxial, Cfootprints:SO-239, symbol CA16:Conn_Coaxial
- added K2, K3, K4: ~, Footprints:Relay_DPDT_Schrack-RT2-FormC_RM5mm, symbol CA16:Rele_2Conm
- D1, D2, D3, D4, D5, D6: symbol schematic:D_Filled -> CA16:D_Filled
- D10, D11, D12, D7, D8, D9: symbol schematic:LED_Filled -> CA16:LED_Filled
- J1, J5: footprint Footprints:PL_PanelMount -> Cfootprints:SO-239; symbol schematic:Conn_Coaxial -> CA16:Conn_Coaxial
- J4: renamed from J2; symbol schematic:Screw_Terminal_01x07 -> CA16:Screw_Terminal_01x07
- J7: renamed from J6; footprint Footprints:PL_PanelMount -> Cfootprints:SO-239; symbol schematic:Conn_Coaxial -> CA16:Conn_Coaxial
- K1, K5, K6: symbol schematic:Rele_2Conm -> CA16:Rele_2Conm
- R1, R2, R3, R4, R5, R6: symbol schematic:R -> CA16:R
Connections:
- net Antena-2: now also K2.A2
- net Antena-3: now also K3.A2
- net Antena-4: now also K4.A2
- net RF_{IN}: now also K2.14, K2.24, K3.14, K3.24, K4.14, K4.24
- net RF_{antena-2}: now also J2.1 (In), K2.11, K2.21
- net RF_{antena-3}: now also J3.1 (In), K3.11, K3.21
- net RF_{antena-4}: now also J6.1 (In), K4.11, K4.21
- net RF_{antena-6}: now also J8.1 (In)
- net GND renamed GND1
- net GND1: now also J2.2 (Ext), J3.2 (Ext), J6.2 (Ext), J8.2 (Ext), K2.12, K2.22, K2.A1, K3.12, K3.22, K3.A1, K4.12, K4.22, K4.A1
